Commit message: Add a floating button Add gravity effect to the door

File: urdf/skew-box-button.urdf (robot description, URDF)
Before this commit: robot skew_box, 10 links, 9 joints
Links:
- link button: mass 0.1 -> 0.01; geometry collision cylinder length=0.05 radius=0.02; visual cylinder length=0.05 radius=0.05
- link door: mass 1 -> 0.1; geometry collision box size=0.16 0.2 0.01; visual box size=0.16 0.2 0.01
- link h1: mass 0.1 -> 0.05
- link h2: mass 0.1 -> 0.05
- link h3: geometry collision cylinder length=0.1 radius=0.01; visual cylinder length=0.1 radius=0.01
Joints:
- joint base_door: limit lower=0 upper=2.5 effort=150.0 velocity=1000 -> lower=0 upper=2.5 effort=0 velocity=0
- joint button_base: axis 0 0 0 -> 0 0 1; limit (none) -> lower=-0.05 upper=0; origin xyz=0 0 0.015 rpy=0 0 0 -> xyz=0 0 0.06 rpy=0 0 0; type fixed -> prismatic

Commit message: Make changes in case of penetrating

File: urdf/skew-box-button.urdf (robot description, URDF)
Before this commit: robot skew_box, 10 links, 9 joints
Links:
- link button: geometry collision cylinder length=0.05 radius=0.02; visual cylinder length=0.03 radius=0.05
Joints:
- joint base_door: limit lower=0 upper=2.5 effort=0 velocity=0 -> lower=0 upper=2 effort=0 velocity=0
- joint button_base: origin xyz=0 0 0.06 rpy=0 0 0 -> xyz=0 0 0.07 rpy=0 0 0
