Commit message: Set the origin of the UR5 arms to be [0 0 0]

File: urdf/ur5_robotiq_140.urdf (robot description, URDF)
Before this commit: robot ur5_robotiq_140, 20 links, 19 joints
Joints:
- joint world_arm_joint: origin xyz=0 0 0.78 rpy=0.0 0.0 0 -> xyz=0 0 0 rpy=0.0 0.0 0

File: urdf/ur5_robotiq_85.urdf (robot description, URDF)
Before this commit: robot ur5_robotiq_85, 20 links, 19 joints
Joints:
- joint world_arm_joint: origin xyz=0 0 0.78 rpy=0.0 0.0 0 -> xyz=0 0 0 rpy=0.0 0.0 0
